File: PCB/_autosave-sennotron.kicad_pcb (KiCad board)
At the start: 2 copper layers, 30 parts, among them J1 Barrel_Jack, J3 Conn_02x08_Odd_Even, J4 Conn_01x16_Female, J5 Screw_Terminal_01x04, J6 Screw_Terminal_01x16, J7 Conn_01x04_Male, J8 Conn_01x04_Male, J9 Conn_01x05_Female, U1 LM1117-3.3, U2 MCP3208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

Commit message: Schematics and PCB design updated
Parts:
- removed J8: Conn_01x04_Male, Pin_Headers:Pin_Header_Straight_1x02_Pitch2.54mm
- added J2: Raspberry_Pi_2_3, Pin_Headers:Pin_Header_Straight_2x20_Pitch2.54mm, F.Cu at (119.4, 38.1)
- D1: value D_Bridge_+-AA -> D_Bridge_+AA-
- J1: footprint custom:CUI-PJ-102A_dc-barrel-jack -> Connectors:BARREL_JACK
- J7: value Conn_01x04_Male -> Conn_02x04_Odd_Even; footprint Pin_Headers:Pin_Header_Straight_1x02_Pitch2.54mm -> Pin_Headers:Pin_Header_Straight_2x04_Pitch2.54mm
- moved J5 91.0 mm to (236.2, 129.2), turned to 90 degrees
- moved R1 89.7 mm to (214.6, 44.5), turned to 270 degrees
- moved J9 87.5 mm to (95.2, 35.6)
- moved R4 86.5 mm to (228.6, 72.4), turned to 270 degrees
- moved R5 82.0 mm to (228.6, 87.6), turned to 270 degrees
- moved U4 73.9 mm to (212.1, 67.3), turned to 90 degrees
- moved D1 72.6 mm to (220.9, 109.2)
- moved C4 72.5 mm to (220.7, 97.8)
- moved R2 71.5 mm to (212.1, 72.4), turned to 270 degrees
- moved U3 69.2 mm to (215.9, 120.7), turned to 180 degrees
- moved R6 69.1 mm to (87.6, 72.4)
- moved R3 65.9 mm to (212.1, 87.6), turned to 270 degrees
- moved C2 64.3 mm to (90.2, 132.2), turned to 270 degrees
- moved J4 61.9 mm to (87.6, 94.0), turned to 90 degrees
- moved J1 58.6 mm to (92.4, 121.9)
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Connections:
- net 3v3_A renamed +3.3VA
- net 5v0 renamed +5V
- D1 pad 2: Net-(C4-Pad2) -> Net-(D1-Pad2)
- D1 pad 4: Net-(D1-Pad4) -> Net-(C4-Pad2)
- J4 pad 10: (no net) -> Net-(J4-Pad10)
- J4 pad 11: (no net) -> lcd_d4
- J4 pad 12: (no net) -> lcd_d5
- J4 pad 13: (no net) -> lcd_d6
- J4 pad 14: (no net) -> lcd_d7
- J4 pad 4: (no net) -> lcd_rs
- J4 pad 6: (no net) -> lcd_en
- J4 pad 7: (no net) -> Net-(J4-Pad7)
- J4 pad 8: (no net) -> Net-(J4-Pad8)
- J4 pad 9: (no net) -> Net-(J4-Pad9)
- J5 pad 2: Net-(D1-Pad4) -> Net-(D1-Pad2)
- J6 pad 1: Net-(J3-Pad2) -> GND
- J6 pad 10: GND -> Net-(J3-Pad8)
- J6 pad 11: Net-(J3-Pad12) -> GND
- J6 pad 12: GND -> Net-(J3-Pad6)
- J6 pad 13: Net-(J3-Pad14) -> GND
- J6 pad 14: GND -> Net-(J3-Pad4)
- J6 pad 15: Net-(J3-Pad16) -> GND
- J6 pad 16: GND -> Net-(J3-Pad2)
- J6 pad 2: GND -> Net-(J3-Pad16)
- J6 pad 3: Net-(J3-Pad4) -> GND
- J6 pad 4: GND -> Net-(J3-Pad14)
- J6 pad 5: Net-(J3-Pad6) -> GND
- J6 pad 6: GND -> Net-(J3-Pad12)
- J6 pad 7: Net-(J3-Pad8) -> GND
- J6 pad 8: GND -> Net-(J3-Pad10)
- J6 pad 9: Net-(J3-Pad10) -> GND
- J7 pad 1: GND -> Net-(J7-Pad1)
- J7 pad 2: Net-(J7-Pad2) -> GND
- J9 pad 3: (no net) -> sda
- J9 pad 4: (no net) -> scl
- J9 pad 5: (no net) -> Net-(J9-Pad5)
- R1 pad 1: 3v3 -> +3V3
- R10 pad 1: Net-(J8-Pad1) -> Net-(J7-Pad6)
- R10 pad 2: (no net) -> btn_2
- R11 pad 1: Net-(J8-Pad4) -> Net-(J7-Pad8)
- R12 pad 2: Net-(J8-Pad1) -> Net-(J7-Pad6)
- R13 pad 2: (no net) -> heat_trig
- R7 pad 1: (no net) -> Net-(J7-Pad1)
- R7 pad 2: (no net) -> led_1
- R8 pad 1: Net-(J7-Pad2) -> Net-(J7-Pad3)
- R8 pad 2: (no net) -> led_2
- R9 pad 1: Net-(J8-Pad4) -> Net-(J7-Pad8)
- R9 pad 2: (no net) -> btn_1
- U2 pad 10: (no net) -> spi_cs_0
- U2 pad 11: (no net) -> spi_mosi
- U2 pad 12: (no net) -> spi_miso
- U2 pad 13: (no net) -> spi_clk
- U2 pad 16: 3v3 -> +3V3
- U4 pad 3: (no net) -> Net-(U4-Pad3)
- U4 pad 6: (no net) -> Net-(U4-Pad6)
Routing:
- net GND: track 0.00 -> 490.2 mm
- net +3V3: track 0.00 -> 193.0 mm
- net +5V: track 0.00 -> 171.4 mm
- net spi_cs_0: track 0.00 -> 109.2 mm
- net spi_mosi: track 0.00 -> 98.3 mm
- net spi_miso: track 0.00 -> 94.8 mm
- net lcd_rs: track 0.00 -> 93.4 mm
- net spi_clk: track 0.00 -> 91.1 mm
- net +3.3VA: track 0.00 -> 90.3 mm
- net heat_trig: track 0.00 -> 83.3 mm
- net lcd_en: track 0.00 -> 81.4 mm
- net btn_1: track 0.00 -> 76.6 mm
- net btn_2: track 0.00 -> 74.0 mm
- net lcd_d4: track 0.00 -> 73.8 mm
- net AC_sens: track 0.00 -> 69.3 mm
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