File: PCB/_saved_sennotron.sch (KiCad schematic (older format))
At the start: 31 parts, among them J1 Barrel_Jack, J2 Raspberry_Pi_2_3, J3 Conn_02x08_Odd_Even, J4 Conn_01x16_Female, J5 Screw_Terminal_01x04, J6 Screw_Terminal_01x16, J7 Conn_01x04_Female, J8 Conn_01x04_Female, J9 Conn_01x05_Female, U1 LM1117-3.3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

Commit message: Schematics and PCB design updated
Parts:
- removed J7, J8: Conn_01x04_Female, Socket_Strips:Socket_Strip_Straight_1x04_Pitch2.54mm, symbol Conn_01x04_Female
- added J7: Conn_02x04_Odd_Even, Pin_Headers:Pin_Header_Straight_2x04_Pitch2.54mm, symbol Conn_02x04_Odd_Even
- D1: footprint custom:CUI-PJ-102A_dc-barrel-jack -> custom:SIP-4
Connections:
- wire segments 82 -> 83
Other:
- moved on the sheet: R10, R11, R12, R9
Changed lines of the file:
@@
 L Screw_Terminal_01x16 J6
 U 1 1 5B031CB2
-P 5400 900
-F 0 "J6" H 5400 1700 50  0000 C CNN
-F 1 "Screw_Terminal_01x16" H 5400 0   50  0000 C CNN
-F 2 "TerminalBlocks_Phoenix:TerminalBlock_Phoenix_PT-3.5mm_16pol" H 5400 900 50  0001 C CNN
-F 3 "" H 5400 900 50  0001 C CNN
-	1    5400 900
-	0    -1   -1   0
+P 5500 900
+F 0 "J6" H 5500 1700 50  0000 C CNN
+F 1 "Screw_Terminal_01x16" H 5500 0   50  0000 C CNN
+F 2 "TerminalBlocks_Phoenix:TerminalBlock_Phoenix_PT-3.5mm_16pol" H 5500 900 50  0001 C CNN
+F 3 "" H 5500 900 50  0001 C CNN
+	1    5500 900
+	0    1    -1   0
 $EndComp
 $Comp
@@
 L R R9
 U 1 1 5B03B02B
-P 7050 4200
-F 0 "R9" V 7130 4200 50  0000 C CNN
-F 1 "R" V 7050 4200 50  0000 C CNN
-F 2 "Resistors_THT:R_Axial_DIN0207_L6.3mm_D2.5mm_P10.16mm_Horizontal" V 6980 4200 50  0001 C CNN
-F 3 "" H 7050 4200 50  0001 C CNN
-	1    7050 4200
-	0    1    1    0
+P 7600 4800
+F 0 "R9" V 7680 4800 50  0000 C CNN
+F 1 "R" V 7600 4800 50  0000 C CNN
+F 2 "Resistors_THT:R_Axial_DIN0207_L6.3mm_D2.5mm_P10.16mm_Horizontal" V 7530 4800 50  0001 C CNN
+F 3 "" H 7600 4800 50  0001 C CNN
+	1    7600 4800
+	1    0    0    -1
 $EndComp
 $Comp
 L R R10
 U 1 1 5B03B074
-P 7050 4800
-F 0 "R10" V 7130 4800 50  0000 C CNN
-F 1 "R" V 7050 4800 50  0000 C CNN
-F 2 "Resistors_THT:R_Axial_DIN0207_L6.3mm_D2.5mm_P10.16mm_Horizontal" V 6980 4800 50  0001 C CNN
-F 3 "" H 7050 4800 50  0001 C CNN
-	1    7050 4800
-	0    1    1    0
+P 8200 4800
+F 0 "R10" V 8280 4800 50  0000 C CNN
+F 1 "R" V 8200 4800 50  0000 C CNN
+F 2 "Resistors_THT:R_Axial_DIN0207_L6.3mm_D2.5mm_P10.16mm_Horizontal" V 8130 4800 50  0001 C CNN
+F 3 "" H 8200 4800 50  0001 C CNN
+	1    8200 4800
+	1    0    0    -1
 $EndComp
 $Comp
 L R R11
 U 1 1 5B03B127
-P 7300 4350
-F 0 "R11" V 7380 4350 50  0000 C CNN
-F 1 "R" V 7300 4350 50  0000 C CNN
-F 2 "Resistors_THT:R_Axial_DIN0207_L6.3mm_D2.5mm_P10.16mm_Horizontal" V 7230 4350 50  0001 C CNN
-F 3 "" H 7300 4350 50  0001 C CNN
-	1    7300 4350
-	1    0    0    -1
+P 7750 4550
+F 0 "R11" V 7830 4550 50  0000 C CNN
+F 1 "R" V 7750 4550 50  0000 C CNN
+F 2 "Resistors_THT:R_Axial_DIN0207_L6.3mm_D2.5mm_P10.16mm_Horizontal" V 7680 4550 50  0001 C CNN
+F 3 "" H 7750 4550 50  0001 C CNN
+	1    7750 4550
+	0    -1   -1   0
 $EndComp
 $Comp
 L GND #PWR018
 U 1 1 5B03B226
-P 7200 4500
-F 0 "#PWR018" H 7200 4250 50  0001 C CNN
-F 1 "GND" H 7200 4350 50  0000 C CNN
-F 2 "" H 7200 4500 50  0001 C CNN
-F 3 "" H 7200 4500 50  0001 C CNN
-	1    7200 4500
-	0    1    1    0
+P 7900 4650
+F 0 "#PWR018" H 7900 4400 50  0001 C CNN
+F 1 "GND" H 7900 4500 50  0000 C CNN
+F 2 "" H 7900 4650 50  0001 C CNN
+F 3 "" H 7900 4650 50  0001 C CNN
+	1    7900 4650
+	1    0    0    -1
 $EndComp
 $Comp
 L R R12
 U 1 1 5B03B270
-P 7300 4650
-F 0 "R12" V 7380 4650 50  0000 C CNN
-F 1 "R" V 7300 4650 50  0000 C CNN
-F 2 "Resistors_THT:R_Axial_DIN0207_L6.3mm_D2.5mm_P10.16mm_Horizontal" V 7230 4650 50  0001 C CNN
-F 3 "" H 7300 4650 50  0001 C CNN
-	1    7300 4650
-	1    0    0    -1
-$EndComp
-Wire Wire Line
-	7300 4500 7200 4500
-Wire Wire Line
-	7650 4450 7650 4550
-Wire Wire Line
-	7200 4200 7650 4200
-Wire Wire Line
-	7650 4200 7650 4350
-Wire Wire Line
-	7200 4800 7650 4800
-Wire Wire Line
-	7650 4800 7650 4650
-Text GLabel 6900 4200 0    39   Input ~ 0
+P 8050 4550
+F 0 "R12" V 8130 4550 50  0000 C CNN
+F 1 "R" V 8050 4550 50  0000 C CNN
+F 2 "Resistors_THT:R_Axial_DIN0207_L6.3mm_D2.5mm_P10.16mm_Horizontal" V 7980 4550 50  0001 C CNN
+F 3 "" H 8050 4550 50  0001 C CNN
+	1    8050 4550
+	0    -1   -1   0
+$EndComp
+Wire Wire Line
+	7900 4550 7900 4650
+Wire Wire Line
+	7600 4100 7600 4650
+Wire Wire Line
+	8200 3800 8200 4650
+Text GLabel 7600 4950 3    39   Input ~ 0
 btn_1
-Text GLabel 6900 4800 0    39   Input ~ 0
+Text GLabel 8200 4950 3    39   Input ~ 0
 btn_2
 Wire Wire Line
 	7200 3600 7650 3600
 Wire Wire Line
-	7200 3800 7650 3800
+	7200 3800 7250 3800
 $Comp
 L GND #PWR019
 U 1 1 5B03B9C8
-P 7650 3700
-F 0 "#PWR019" H 7650 3450 50  0001 C CNN
-F 1 "GND" H 7650 3550 50  0000 C CNN
-F 2 "" H 7650 3700 50  0001 C CNN
-F 3 "" H 7650 3700 50  0001 C CNN
-	1    7650 3700
-	0    1    1    0
+P 8150 3600
+F 0 "#PWR019" H 8150 3350 50  0001 C CNN
+F 1 "GND" H 8150 3450 50  0000 C CNN
+F 2 "" H 8150 3600 50  0001 C CNN
+F 3 "" H 8150 3600 50  0001 C CNN
+	1    8150 3600
+	0    -1   -1   0
 $EndComp
 $Comp
 L GND #PWR020
 U 1 1 5B03BA18
-P 7650 3900
-F 0 "#PWR020" H 7650 3650 50  0001 C CNN
-F 1 "GND" H 7650 3750 50  0000 C CNN
-F 2 "" H 7650 3900 50  0001 C CNN
-F 3 "" H 7650 3900 50  0001 C CNN
-	1    7650 3900
-	0    1    1    0
+P 8150 3700
+F 0 "#PWR020" H 8150 3450 50  0001 C CNN
+F 1 "GND" H 8150 3550 50  0000 C CNN
+F 2 "" H 8150 3700 50  0001 C CNN
+F 3 "" H 8150 3700 50  0001 C CNN
+	1    8150 3700
+	0    -1   -1   0
 $EndComp
 Text GLabel 6800 3600 0    39   Input ~ 0
@@
 Connection ~ 2650 5650
 Connection ~ 3050 5650
-Connection ~ 7300 4200
-Connection ~ 7300 4800
+Connection ~ 7600 4550
+Connection ~ 8200 4550
 Text GLabel 9200 4550 0    39   Input ~ 0
 heat_trig
@@
 L +3.3V #PWR034
 U 1 1 5B04ABE7
-P 7600 4500
-F 0 "#PWR034" H 7600 4350 50  0001 C CNN
-F 1 "+3.3V" H 7600 4640 50  0000 C CNN
-F 2 "" H 7600 4500 50  0001 C CNN
-F 3 "" H 7600 4500 50  0001 C CNN
-	1    7600 4500
-	0    -1   -1   0
-$EndComp
-Wire Wire Line
-	7650 4500 7600 4500
-Connection ~ 7650 4500
+P 7650 3900
+F 0 "#PWR034" H 7650 3750 50  0001 C CNN
+F 1 "+3.3V" H 7650 4040 50  0000 C CNN
+F 2 "" H 7650 3900 50  0001 C CNN
+F 3 "" H 7650 3900 50  0001 C CNN
+	1    7650 3900
+	0    -1   -1   0
+$EndComp
 NoConn ~ 9850 1600
 $Comp
@@
 F 0 "D1" H 10000 3825 50  0000 L CNN
 F 1 "D_Bridge_+AA-" H 10000 3750 50  0000 L CNN
-F 2 "custom:CUI-PJ-102A_dc-barrel-jack" H 9950 3550 50  0001 C CNN
+F 2 "custom:SIP-4" H 9950 3550 50  0001 C CNN
 F 3 "" H 9950 3550 50  0001 C CNN
 	1    9950 3550
@@
 $EndComp
 $Comp
-L Conn_01x04_Female J7
-U 1 1 5B0575FF
+L Conn_02x04_Odd_Even J7
+U 1 1 5B057DD3
 P 7850 3700
-F 0 "J7" H 7850 3900 50  0000 C CNN
-F 1 "Conn_01x04_Female" H 7850 3400 50  0000 C CNN
-F 2 "Socket_Strips:Socket_Strip_Straight_1x04_Pitch2.54mm" H 7850 3700 50  0001 C CNN
+F 0 "J7" H 7900 3900 50  0000 C CNN
+F 1 "Conn_02x04_Odd_Even" H 7900 3400 50  0000 C CNN
+F 2 "Pin_Headers:Pin_Header_Straight_2x04_Pitch2.54mm" H 7850 3700 50  0001 C CNN
 F 3 "" H 7850 3700 50  0001 C CNN
 	1    7850 3700
 	1    0    0    -1
 $EndComp
-$Comp
-L Conn_01x04_Female J8
-U 1 1 5B057676
-P 7850 4450
-F 0 "J8" H 7850 4650 50  0000 C CNN
-F 1 "Conn_01x04_Female" H 7850 4150 50  0000 C CNN
-F 2 "Socket_Strips:Socket_Strip_Straight_1x04_Pitch2.54mm" H 7850 4450 50  0001 C CNN
-F 3 "" H 7850 4450 50  0001 C CNN
-	1    7850 4450
-	1    0    0    -1
-$EndComp
+Wire Wire Line
+	7650 3700 7250 3700
+Wire Wire Line
+	7250 3700 7250 3800
+Connection ~ 7250 3800
+$Comp
+L +3.3V #PWR047
+U 1 1 5B0589A8
+P 7650 3800
+F 0 "#PWR047" H 7650 3650 50  0001 C CNN
+F 1 "+3.3V" H 7650 3940 50  0000 C CNN
+F 2 "" H 7650 3800 50  0001 C CNN
+F 3 "" H 7650 3800 50  0001 C CNN
+	1    7650 3800
+	0    -1   -1   0
+$EndComp
+Wire Wire Line
+	8150 3900 8150 4100
+Wire Wire Line
+	8150 4100 7600 4100
+Wire Wire Line
+	8200 3800 8150 3800
 $EndSCHEMATC
