File: PCB/sennotron - Kopie.sch (KiCad schematic (older format))
At the start: 31 parts, among them J1 Barrel_Jack, J2 Raspberry_Pi_2_3, J3 Conn_02x08_Odd_Even, J4 Conn_01x16_Female, J5 Screw_Terminal_01x04, J6 Screw_Terminal_01x16, J7 Conn_01x04_Female, J8 Conn_01x04_Female, J9 Conn_01x05_Female, U1 LM1117-3.3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

Commit message: Schematics and PCB design updated
Parts:
- removed D1: D_Bridge_+AA-, custom:CUI-PJ-102A_dc-barrel-jack, symbol D_Bridge_+AA-
- removed J7, J8: Conn_01x04_Female, Socket_Strips:Socket_Strip_Straight_1x04_Pitch2.54mm, symbol Conn_01x04_Female
- added D1: D_Bridge_+-AA, custom:SIP-4, symbol D_Bridge_+-AA
- added J10: Conn_02x20_Odd_Even, Pin_Headers:Pin_Header_Straight_2x20_Pitch2.54mm, symbol Conn_02x20_Odd_Even
- added J7, J8: Conn_01x04_Male, Pin_Headers:Pin_Header_Straight_1x02_Pitch2.54mm, symbol Conn_01x04_Male
Connections:
- wire segments 82 -> 86
- no-connect marks 17 -> 27
Other:
- moved on the sheet: J2
