File: PCB/_saved_sennotron_2.sch (KiCad schematic (older format))
At the start: 32 parts, among them J1 Barrel_Jack, J10 Conn_02x20_Odd_Even, J2 Raspberry_Pi_2_3, J3 Conn_02x08_Odd_Even, J4 Conn_01x16_Female, J5 Screw_Terminal_01x02, J6 Screw_Terminal_01x16, J7 Conn_01x04_Male, J8 Conn_01x04_Male, J9 Conn_01x05_Female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

Commit message: pcb design almost done... waiting for a review!
Parts:
- removed J1: Barrel_Jack, Connectors:BARREL_JACK, symbol Barrel_Jack
- removed J5: Screw_Terminal_01x02, TerminalBlocks_Phoenix:TerminalBlock_Phoenix_PT-3.5mm_2pol, symbol Screw_Terminal_01x02
- removed J7, J8: Conn_01x04_Male, Pin_Headers:Pin_Header_Straight_1x04_Pitch2.54mm, symbol Conn_01x04_Male
- added J1: Screw_Terminal_01x02, TerminalBlocks_Phoenix:TerminalBlock_Phoenix_PT-3.5mm_2pol, symbol Screw_Terminal_01x02
- added J11, J12, J13, J14, J15, J16, J17, J18, J19, J8: Conn_01x01, custom:Pad_2.5, symbol Conn_01x01
- added J5: Conn_02x04_Odd_Even, Pin_Headers:Pin_Header_Straight_2x04_Pitch2.54mm, symbol Conn_02x04_Odd_Even
- added J7: Screw_Terminal_01x04, TerminalBlocks_Phoenix:TerminalBlock_Phoenix_PT-3.5mm_4pol, symbol Screw_Terminal_01x04
- added R14: R, Resistors_THT:R_Axial_DIN0207_L6.3mm_D2.5mm_P10.16mm_Horizontal, symbol R
- added U5: S102S01, Housings_SIP:SIP4_Sharp-SSR_Pitch7.62mm_Straight, symbol S102S01
- J10: footprint Pin_Headers:Pin_Header_Straight_2x20_Pitch2.54mm -> custom:raspberry_pi_zero
- J6: footprint TerminalBlocks_Phoenix:TerminalBlock_Phoenix_PT-3.5mm_16pol -> custom:springlock
Connections:
- net labels removed: 220L, 220N, btn, lcd, lcd1, lcd2, lcd3, lcd4, lcd5, lcd6, led, ledbtn
- wire segments 140 -> 159
- no-connect marks 29 -> 32
Other:
- note removed: "lcd_d4"
- note removed: "lcd_d5"
- note removed: "lcd_d6"
- note removed: "lcd_d7"
- note removed: "lcd_en"
- note removed: "lcd_rs"
- moved on the sheet: D1, J10, J3, J4, J6, J9, R10, R11, R12, R6, R7, R8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
