File: PCB/sennotron_2.sch (KiCad schematic (older format))
At the start: 32 parts, among them J1 Barrel_Jack, J10 Conn_02x20_Odd_Even, J2 Raspberry_Pi_2_3, J3 Conn_02x08_Odd_Even, J4 Conn_01x16_Female, J5 Screw_Terminal_01x02, J6 Screw_Terminal_01x16, J7 Conn_01x04_Male, J8 Conn_01x04_Male, J9 Conn_01x05_Female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

Commit message: pcb design almost done... waiting for a review!
Parts:
- removed J1: Barrel_Jack, Connectors:BARREL_JACK, symbol Barrel_Jack
- added J?: Screw_Terminal_01x02, TerminalBlocks_Phoenix:TerminalBlock_Phoenix_PT-3.5mm_2pol, symbol Screw_Terminal_01x02
- added L?: L, symbol L
- added SW? (x2): SW_Push, symbol SW_Push
- added U? (x2): S102S01, Housings_SIP:SIP4_Sharp-SSR_Pitch7.62mm_Straight, symbol S102S01
Connections:
- net lcd1 is gone; now on net lcd_rs: J10.22 (Pin_22), J4.4 (Pin_4)
- net lcd2 is gone; now on net lcd_en: J10.18 (Pin_18), J4.6 (Pin_6)
- net lcd3 is gone; now on net lcd_d4: J10.16 (Pin_16), J4.11 (Pin_11)
- net lcd4 is gone; now on net lcd_d5: J10.12 (Pin_12), J4.12 (Pin_12)
- net lcd5 is gone; now on net lcd_d6: J10.10 (Pin_10), J4.13 (Pin_13)
- net lcd6 is gone; now on net lcd_d7: J10.8 (Pin_8), J4.14 (Pin_14)
- net +5V: now also J?.2 (Pin_2)
- net GND: now also J?.1 (Pin_1), SW?.2, U?.1
- net 220N: now reaches D1.4, J5.1 (Pin_1)
- net 220N: now also U3.2; no longer U3.1
- net 220L: now reaches D1.3, J5.2 (Pin_2)
- net 220L: now also U3.1; no longer U3.2
- new net: L?.2, SW?.2, U?.1
- new net: L?.1, SW?.1, U?.2
- new net VAC: SW?.1, U?.2
- no-connect marks 29 -> 28
Other:
- note removed: "lcd_d4"
- note removed: "lcd_d5"
- note removed: "lcd_d6"
- note removed: "lcd_d7"
- note removed: "lcd_en"
- note removed: "lcd_rs"
- moved on the sheet: R6, U2
